File: RasPi_NFC_Audio_KiCAD/RasPi_NFC_Audio_KiCAD.kicad_pcb (KiCad board)
At the start: 2 copper layers, 116 x 65 mm, 74 parts, among them J1 Barrel_Jack_Switch, J2 Conn_02x20_Odd_Even, J3 Connector_01x10, J4 Screw_Terminal_01x02, J5 Screw_Terminal_01x02, U1 MIC5225-3.3V, U2 PN532, U3 MAX98357, U4 MAX98357, Y1 Oscillator

Commit message: Layout updates
Parts:
- J1, J3, J4, J5, U3, U4: moved to B.Cu
- moved J3 24.9 mm to (131.2, 27.5), turned to 180 degrees
- moved C15 22.1 mm to (110.4, 49.3), turned to 180 degrees
- moved R6 20.9 mm to (112.3, 52.8), turned to 180 degrees
- moved J1 20.4 mm to (104.0, 86.0), turned to 0 degrees
- moved J4 19.7 mm to (109.1, 27.5)
- moved U1 19.0 mm to (128.0, 67.0)
- moved C17 18.5 mm to (109.2, 56.8), turned to 180 degrees
- moved U3 14.1 mm to (112.2, 36.4), turned to 90 degrees
- moved TP8 13.7 mm to (85.4, 27.4)
- moved TP7 11.3 mm to (92.2, 27.6)
- moved TP1 11.3 mm to (120.3, 94.6)
- moved J5 10.1 mm to (100.7, 27.4)
- moved MK3 10.0 mm to (42.2, 26.7)
- moved MK4 10.0 mm to (42.2, 84.7)
- moved R7 9.48 mm to (109.6, 62.7)
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Other:
- board size 116 x 65 mm -> 106 x 65 mm

Commit message: Layout updates
Parts:
- C15, C17, C18, C19, C20, C21, C22, C23, J1, J2, J3, J4, J5, L1, L2, R6, R7, R8, R9, U2, U3, U4, Y1: moved to F.Cu
- R10, R11: moved to B.Cu
- moved J2 48.2 mm to (139.9, 79.8)
- moved J3 41.6 mm to (157.6, 59.7)
- moved TP6 10.9 mm to (125.8, 27.8)
- moved TP5 10.1 mm to (130.2, 28.1)
- moved R10 6.43 mm to (94.9, 60.2), turned to 90 degrees
- moved R11 6.13 mm to (94.9, 53.9), turned to 90 degrees
- moved J1 5.31 mm to (109.3, 86.0), turned to 180 degrees
- moved J4 2.77 mm to (111.9, 27.5)
- moved J5 0.28 mm to (100.4, 27.6)
- turned C18 to 90 degrees
- turned C19 to 90 degrees
- turned C20 to 90 degrees
- turned C21 to 90 degrees
- turned R8 to 90 degrees
- turned R9 to 90 degrees
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
Commit message: Layout updates
Parts:
- moved R15 122.0 mm to (103.2, 44.9)
- moved R16 121.9 mm to (120.3, 31.9), turned to 180 degrees
- moved R17 121.0 mm to (106.9, 41.5), turned to 180 degrees
- moved R14 121.0 mm to (103.2, 41.5), turned to 180 degrees
- moved C26 120.4 mm to (123.1, 25.7), turned to 90 degrees
- moved C27 119.2 mm to (110.4, 39.1)
- moved C24 117.8 mm to (123.1, 30.1), turned to 270 degrees
- moved R12 117.3 mm to (116.5, 31.9), turned to 180 degrees
- moved C25 117.2 mm to (110.4, 35.6)
- moved R13 116.8 mm to (116.4, 35.0), turned to 180 degrees
- moved TP4 113.0 mm to (92.1, 52.8)
- moved TP3 110.2 mm to (92.2, 62.8)
- moved C8 95.1 mm to (117.0, 47.5), turned to 180 degrees
- moved C13 84.7 mm to (114.8, 60.3), turned to 270 degrees
- moved C11 82.9 mm to (116.9, 53.7), turned to 180 degrees
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Other:
- board size 106 x 65 mm -> 103.5 x 65 mm

Commit message: Layout updates
Parts:
- J2: footprint Connector_PinSocket_2.54mm:PinSocket_2x20_P2.54mm_Vertical -> Connector_PinHeader_2.54mm:PinHeader_2x20_P2.54mm_Vertical
- TP3: value TestPoint -> ANT-; footprint TestPoint:TestPoint_Pad_2.0x2.0mm -> TestPoint:TestPoint_Pad_1.0x1.0mm
- TP4: value TestPoint -> ANT+; footprint TestPoint:TestPoint_Pad_2.0x2.0mm -> TestPoint:TestPoint_Pad_1.0x1.0mm
- moved J2 48.2 mm to (140.1, 31.5), turned to 0 degrees
- moved C22 14.3 mm to (104.2, 50.5), turned to 90 degrees
- moved R6 14.1 mm to (114.9, 66.8)
- moved C23 14.1 mm to (104.2, 64.6), turned to 90 degrees
- moved C15 14.0 mm to (114.9, 63.8)
- moved C19 13.5 mm to (108.4, 50.6)
- moved C20 13.1 mm to (108.4, 64.6)
- moved C17 7.27 mm to (111.4, 64.7), turned to 90 degrees
- moved R7 7.06 mm to (109.3, 56.8), turned to 180 degrees
- moved L2 5.85 mm to (109.3, 60.5)
- moved L1 5.64 mm to (109.3, 54.8)
- moved R5 5.47 mm to (130.8, 60.2), turned to 0 degrees
- moved C21 4.25 mm to (105.6, 59.6)
- moved C18 4.18 mm to (105.6, 55.7)
- moved R9 4.11 mm to (102.9, 59.6)
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Routing:
- net NFC_RST_PDN_N: track 0.00 -> 36.4 mm, vias 0 -> 2
- net NFC_RSTOUT_N: track 0.00 -> 27.1 mm, vias 0 -> 1
- net NFC_IRQ: track 0.00 -> 27.0 mm
- net SEL1: track 0.00 -> 14.9 mm
- net Net-(C17-Pad1): track 0.00 -> 13.0 mm
- net SEL0: track 0.00 -> 11.8 mm
- net GND: track 5.32 -> 16.4 mm
- net Net-(C6-Pad1): track 0.00 -> 9.43 mm
- net Net-(C21-Pad2): track 0.00 -> 8.82 mm
- net +3V3: track 0.00 -> 8.57 mm
- net Net-(L1-Pad1): track 0.00 -> 8.46 mm
- net VCOM: track 0.00 -> 8.31 mm
- net Net-(C18-Pad2): track 0.00 -> 8.20 mm
- net Net-(C17-Pad2): track 0.00 -> 8.20 mm
- net VCC: track 0.00 -> 8.08 mm
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- added copper zone on B.Cu, net GND
Other:
- rule trace_min: 0.2 -> 0.16
- board text removed: "RASPBERRY-PI 40-PIN ADDON BOARD VIEW FROM TOP NOTE: P1 SHOULD BE FITTED ON THE REVERSE OF THE BOARD ADD EDGE CUTS FROM CAMERA AND DISPLAY PORTS AS REQUIRED"

Commit message: Layout updates
Parts:
- added C28: 100u, Capacitor_SMD:C_1206_3216Metric_Pad1.42x1.75mm_HandSolder, F.Cu at (137.7, 106.4)
- TP3: value ANT- -> TestPoint
- TP4: value ANT+ -> TestPoint
- moved MK3 183.6 mm to (208.5, 109.7), turned to 90 degrees
- moved MK4 167.0 mm to (208.5, 51.7), turned to 90 degrees
- moved TP8 93.7 mm to (174.2, 51.0), turned to 270 degrees
- moved MK1 88.1 mm to (112.0, 109.7), turned to 270 degrees
- moved TP7 85.4 mm to (170.4, 51.0), turned to 270 degrees
- moved J2 78.1 mm to (113.1, 104.9), turned to 180 degrees
- moved TP4 74.5 mm to (160.4, 86.1), turned to 180 degrees
- moved J5 74.4 mm to (165.8, 52.1)
- moved TP3 68.5 mm to (160.3, 77.4), turned to 180 degrees
- moved R11 66.5 mm to (156.3, 85.2), turned to 270 degrees
- moved TP1 65.1 mm to (159.4, 110.1), turned to 270 degrees
- moved TP2 64.4 mm to (154.8, 110.1), turned to 270 degrees
- moved J3 64.3 mm to (95.6, 76.7), turned to 0 degrees
- moved TP6 62.1 mm to (157.7, 51.0), turned to 270 degrees
- moved R10 61.7 mm to (156.3, 78.9), turned to 270 degrees
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Connections:
- TP5 pad 1: Net-(J4-Pad1) -> Net-(J4-Pad2)
- TP6 pad 1: Net-(J4-Pad2) -> Net-(J4-Pad1)
- TP7 pad 1: Net-(J5-Pad1) -> Net-(J5-Pad2)
- TP8 pad 1: Net-(J5-Pad2) -> Net-(J5-Pad1)
- U3 pad 10: Net-(J4-Pad1) -> Net-(J4-Pad2)
- U3 pad 9: Net-(J4-Pad2) -> Net-(J4-Pad1)
- U4 pad 10: Net-(J5-Pad1) -> Net-(J5-Pad2)
- U4 pad 9: Net-(J5-Pad2) -> Net-(J5-Pad1)
Routing:
- net +5V: track 0.00 -> 168.9 mm, vias 0 -> 2
- net I2S_CK: track 0.00 -> 86.9 mm, vias 0 -> 3
- net I2S_WS: track 0.00 -> 51.6 mm, vias 0 -> 4
- net Net-(J5-Pad1): track 0.00 -> 39.4 mm
- net Net-(J5-Pad2): track 0.00 -> 32.4 mm
- net AUDIO_SD_N_0: track 0.00 -> 31.4 mm
- net I2S_SD: track 0.00 -> 29.3 mm
- net PI_UART_RX: track 0.00 -> 22.7 mm, vias 0 -> 2
- net Net-(J4-Pad1): track 0.00 -> 21.7 mm
- net PI_UART_TX: track 0.00 -> 20.4 mm, vias 0 -> 2
- net Net-(J4-Pad2): track 0.00 -> 15.1 mm
- net VCOM: track 8.31 -> 22.3 mm, vias 0 -> 1
- net +3V3: track 8.57 -> 18.2 mm
- net /GPIO14(TXD0): track 0.00 -> 9.47 mm
- net /GPIO15(RXD0): track 0.00 -> 9.20 mm
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Other:
- board size 103.5 x 65 mm -> 104 x 65.3 mm
- board text added: "SPRK-L"
- board text added: "SPRK-R"

Commit message: Layout updates
Parts:
- removed J3: Connector_01x10, Connector_PinHeader_2.54mm:PinHeader_1x10_P2.54mm_Vertical
- moved C3 52.3 mm to (116.8, 79.1)
- moved R15 42.1 mm to (139.4, 65.7)
- moved R17 41.7 mm to (147.9, 70.6), turned to 90 degrees
- moved R14 41.7 mm to (139.6, 68.8)
- moved R16 20.5 mm to (124.7, 63.5), turned to 180 degrees
- moved R4 20.0 mm to (124.9, 111.4), turned to 0 degrees
- moved R13 19.9 mm to (131.3, 59.8), turned to 180 degrees
- moved R3 19.7 mm to (117.7, 111.4), turned to 0 degrees
- moved R12 14.2 mm to (131.3, 57.3)
Routing:
- net GND: track 23.5 -> 128.0 mm, vias 1 -> 31
- net AUDIO_SD_N_1: track 0.00 -> 41.9 mm, vias 0 -> 4
- net +5V: track 168.9 -> 199.5 mm
- net +3V3: track 18.2 -> 48.2 mm, vias 0 -> 3
- net VCOM: track 22.3 -> 43.5 mm
- net I2S_SD: track 29.3 -> 48.5 mm, vias 0 -> 4
- net /GPIO3(SCL1): track 7.20 -> 25.7 mm, vias 0 -> 2
- net Net-(R12-Pad2): track 0.00 -> 11.1 mm, vias 0 -> 2
- net /GPIO2(SDA1): track 7.80 -> 18.2 mm, vias 1 -> 2
- net Net-(R14-Pad2): track 0.00 -> 10.1 mm, vias 0 -> 2
- net I2S_CK: track 86.9 -> 81.3 mm, vias 3 -> 4
- net AUDIO_SD_N_0: track 31.4 -> 35.5 mm

Commit message: Layout updates
Parts:
- removed TP3, TP4: TestPoint, TestPoint:TestPoint_Pad_1.0x1.0mm
- moved R5 0.48 mm to (122.4, 79.5)
Routing:
- net GND: track 128.0 -> 139.3 mm, vias 31 -> 46
- net VCC: track 8.08 -> 19.3 mm, vias 0 -> 3
- net Net-(R10-Pad1): track 384.2 -> 379.8 mm, vias 6 -> 5
- net Net-(R11-Pad2): track 384.0 -> 379.8 mm, vias 4 -> 3
- added copper zone on F.Cu, net GND
Other:
- board size 104 x 65.3 mm -> 103.5 x 65 mm

Commit message: Layout updates
Other:
- board text added: "5V"
- board text added: "GND"
- board text added: "Pi Zero NFC/Audio Skirt"
Changed lines of the file:
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@@
   (general
     (thickness 1.6)
-    (drawings 15)
+    (drawings 19)
     (tracks 782)
     (zones 0)
@@
   )
   (setup
-    (last_trace_width 0.16)
+    (last_trace_width 0.25)
     (user_trace_width 0.16)
     (user_trace_width 0.2)
@@
     (tags "capacitor handsolder")
     (attr smd)
-    (fp_text reference C1 (at 3.3925 -0.1524) (layer F.SilkS)
+    (fp_text reference C1 (at -0.6239 -2.413) (layer F.SilkS)
       (effects (font (size 1 1) (thickness 0.15)))
     )
-    (fp_text value 100u (at 0.6747 -3.1496) (layer F.Fab)
+    (fp_text value 100u (at 1.0271 -3.175) (layer F.Fab)
       (effects (font (size 1 1) (thickness 0.15)))
     )
@@
     (tags "capacitor handsolder")
     (attr smd)
-    (fp_text reference C2 (at 2.4498 0.0762) (layer F.SilkS)
+    (fp_text reference C2 (at 2.653 0.0508) (layer F.SilkS)
       (effects (font (size 1 1) (thickness 0.15)))
     )
@@
     (tags "capacitor handsolder")
     (attr smd)
-    (fp_text reference C5 (at 2.4778 -0.0762) (layer F.SilkS)
+    (fp_text reference C5 (at -0.1892 -1.778) (layer F.SilkS)
       (effects (font (size 1 1) (thickness 0.15)))
     )
-    (fp_text value 10u (at 3.7478 -0.381) (layer F.Fab)
+    (fp_text value 10u (at 2.6048 0.127) (layer F.Fab)
       (effects (font (size 1 1) (thickness 0.15)))
     )
@@
       (effects (font (size 1 1) (thickness 0.15)))
     )
-    (fp_text value 0.1u (at 0 1.43) (layer F.Fab) hide
+    (fp_text value 0.1u (at 0.1384 -1.5494) (layer F.Fab)
       (effects (font (size 1 1) (thickness 0.15)))
     )
@@
       (effects (font (size 1 1) (thickness 0.15)))
     )
-    (fp_text value 10u (at 0 1.43 90) (layer F.Fab) hide
+    (fp_text value 10u (at 0.367 2.413 180) (layer F.Fab)
       (effects (font (size 1 1) (thickness 0.15)))
     )
@@
     (descr "Thin-pin DC Barrel Jack, https://cdn-shop.adafruit.com/datasheets/21mmdcjackDatasheet.pdf")
     (tags "Power Jack")
-    (fp_text reference J1 (at 5.75 8.45 270) (layer F.SilkS)
-      (effects (font (size 1 1) (thickness 0.15)))
+    (fp_text reference J1 (at 3.556 -3.048) (layer F.SilkS)
+      (effects (font (size 1.5 1.5) (thickness 0.15)))
     )
     (fp_text value Barrel_Jack_Switch (at -5.5 6.2 270) (layer F.Fab) hide
@@
       (effects (font (size 1 1) (thickness 0.15)))
     )
-    (fp_text value 10k (at 0 1.43) (layer F.Fab) hide
+    (fp_text value 10k (at -0.1156 -1.5494) (layer F.Fab)
       (effects (font (size 1 1) (thickness 0.15)))
     )
@@
     (tags resistor)
     (attr smd)
-    (fp_text reference R10 (at 1.6256 -1.7526 180) (layer B.SilkS)
+    (fp_text reference R10 (at 0.9652 -2.159 180) (layer B.SilkS)
       (effects (font (size 1 1) (thickness 0.15)) (justify mirror))
     )
-    (fp_text value 0 (at -0.1524 -1.3208 180) (layer B.Fab)
+    (fp_text value 0 (at -0.6858 -1.397 180) (layer B.Fab)
       (effects (font (size 1 1) (thickness 0.15)) (justify mirror))
     )
@@
     (tags resistor)
     (attr smd)
-    (fp_text reference R11 (at 2.4868 -1.4732 180) (layer B.SilkS)
+    (fp_text reference R11 (at 0.785 -2.0066 180) (layer B.SilkS)
       (effects (font (size 1 1) (thickness 0.15)) (justify mirror))
     )
-    (fp_text value 0 (at -0.3072 -1.1176 180) (layer B.Fab)
+    (fp_text value 0 (at -0.739 -1.3716 180) (layer B.Fab)
       (effects (font (size 1 1) (thickness 0.15)) (justify mirror))
     )
@@
     (descr "Through hole straight pin header, 2x20, 2.54mm pitch, double rows")
     (tags "Through hole pin header THT 2x20 2.54mm double row")
-    (fp_text reference J2 (at -2.4892 -2.4638) (layer F.SilkS)
-      (effects (font (size 1 1) (thickness 0.15)))
+    (fp_text reference J2 (at -3.429 48.6156) (layer F.SilkS)
+      (effects (font (size 1.5 1.5) (thickness 0.15)))
     )
     (fp_text value Conn_02x20_Odd_Even (at 1.27 50.59) (layer F.Fab) hide
@@
     )
   )
+  (gr_text GND (at 159.233 106.82) (layer F.SilkS)
+    (effects (font (size 1.2 1.2) (thickness 0.2)))
+  )
+  (gr_text 5V (at 154.915 106.82) (layer F.SilkS)
+    (effects (font (size 1.2 1.2) (thickness 0.2)))
+  )
+  (gr_circle (center 145.136 61.989) (end 145.263 62.116) (layer F.SilkS) (width 0.15))
+  (gr_circle (center 138.151 52.337) (end 138.278 52.464) (layer F.SilkS) (width 0.15))
+  (gr_text "Pi Zero\nNFC/Audio\nSkirt" (at 182.601 80.404) (layer F.SilkS)
+    (effects (font (size 4 4) (thickness 0.6)))
+  )
   (gr_text SPRK-R (at 172.2886 55.1818) (layer F.SilkS)
     (effects (font (size 1.2 1.2) (thickness 0.2)))
@@
   (gr_line (start 208.9654 113.2462) (end 161.4654 113.2462) (layer Edge.Cuts) (width 0.1))
   (gr_line (start 138.9384 48.146) (end 138.9384 113.1192) (layer F.SilkS) (width 0.1))
-  (dimension 30.022897 (width 0.15) (layer B.SilkS)
-    (gr_text "30.023 mm" (at 123.42273 118.799876 -0.1454204479) (layer B.SilkS)
-      (effects (font (size 1 1) (thickness 0.15)))
-    )
-    (feature1 (pts (xy 138.4558 110.2998) (xy 138.435941 118.124399)))
-    (feature2 (pts (xy 108.433 110.2236) (xy 108.413141 118.048199)))
-    (crossbar (pts (xy 108.414629 117.46178) (xy 138.437429 117.53798)))
-    (arrow1a (pts (xy 138.437429 117.53798) (xy 137.30944 118.12154)))
-    (arrow1b (pts (xy 138.437429 117.53798) (xy 137.312417 116.948702)))
-    (arrow2a (pts (xy 108.414629 117.46178) (xy 109.539641 118.051058)))
-    (arrow2b (pts (xy 108.414629 117.46178) (xy 109.542618 116.87822)))
-  )
   (gr_line (start 111.4654 113.2462) (end 127.4654 113.2462) (layer Edge.Cuts) (width 0.1))
   (gr_arc (start 111.4654 51.2462) (end 108.4654 51.2462) (angle 90) (layer Edge.Cuts) (width 0.1))
@@
   (gr_line (start 211.9654 110.2462) (end 211.9654 51.2462) (layer Edge.Cuts) (width 0.1))
   (gr_line (start 127.4654 113.2462) (end 161.4654 113.2462) (layer Edge.Cuts) (width 0.1))
-  (via (at 134.722 81.6994) (size 0.6) (drill 0.4) (layers F.Cu B.Cu) (net 3))
-  (via (at 132.69 81.674) (size 0.6) (drill 0.4) (layers F.Cu B.Cu) (net 3))
-  (via (at 154.153 106.185) (size 0.6) (drill 0.4) (layers F.Cu B.Cu) (net 3))
-  (via (at 153.137 104.915) (size 0.6) (drill 0.4) (layers F.Cu B.Cu) (net 3))
-  (segment (start 154.153 106.185) (end 154.153 105.931) (width 0.25) (layer F.Cu) (net 3))
-  (segment (start 154.153 105.931) (end 153.137 104.915) (width 0.25) (layer F.Cu) (net 3))
-  (segment (start 153.391 59.068) (end 153.264 59.195) (width 0.25) (layer B.Cu) (net 3))
-  (via (at 153.264 59.195) (size 0.6) (drill 0.4) (layers F.Cu B.Cu) (net 3))
-  (via (at 153.391 57.798) (size 0.6) (drill 0.4) (layers F.Cu B.Cu) (net 3))
-  (segment (start 153.391 59.068) (end 153.264 59.195) (width 0.25) (layer F.Cu) (net 3))
-  (segment (start 153.391 57.798) (end 153.391 59.068) (width 0.25) (layer F.Cu) (net 3))
   (segment (start 138.687 86.867) (end 138.673 86.881) (width 0.16) (layer F.Cu) (net 1))
   (segment (start 138.687 84.976) (end 138.687 86.867) (width 0.5) (layer F.Cu) (net 1))
@@
   (segment (start 149.5048 71.0822) (end 149.5048 67.6278) (width 0.16) (layer F.Cu) (net 2))
   (segment (start 149.101 71.486) (end 149.5048 71.0822) (width 0.16) (layer F.Cu) (net 2))
+  (via (at 134.722 81.6994) (size 0.6) (drill 0.4) (layers F.Cu B.Cu) (net 3))
+  (via (at 132.69 81.674) (size 0.6) (drill 0.4) (layers F.Cu B.Cu) (net 3))
+  (via (at 154.153 106.185) (size 0.6) (drill 0.4) (layers F.Cu B.Cu) (net 3))
+  (via (at 153.137 104.915) (size 0.6) (drill 0.4) (layers F.Cu B.Cu) (net 3))
+  (segment (start 154.153 106.185) (end 154.153 105.931) (width 0.25) (layer F.Cu) (net 3))
+  (segment (start 154.153 105.931) (end 153.137 104.915) (width 0.25) (layer F.Cu) (net 3))
+  (segment (start 153.391 59.068) (end 153.264 59.195) (width 0.25) (layer B.Cu) (net 3))
+  (via (at 153.264 59.195) (size 0.6) (drill 0.4) (layers F.Cu B.Cu) (net 3))
+  (via (at 153.391 57.798) (size 0.6) (drill 0.4) (layers F.Cu B.Cu) (net 3))
+  (segment (start 153.391 59.068) (end 153.264 59.195) (width 0.25) (layer F.Cu) (net 3))
+  (segment (start 153.391 57.798) (end 153.391 59.068) (width 0.25) (layer F.Cu) (net 3))
   (via (at 156.312 83.6933) (size 0.6) (drill 0.4) (layers F.Cu B.Cu) (net 3))
   (segment (start 156.312 79.4158) (end 156.312 83.6933) (width 0.2) (layer B.Cu) (net 3))
