File: RasPi_NFC_Audio_KiCAD/RasPi_NFC_Audio_KiCAD.kicad_pcb (KiCad board)
At the start: 2 copper layers, 103.5 x 65 mm, 72 parts, among them J1 Barrel_Jack_Switch, J2 Conn_02x20_Odd_Even, J4 Screw_Terminal_01x02, J5 Screw_Terminal_01x02, U1 MIC5225-3.3V, U2 PN532, U3 MAX98357, U4 MAX98357, Y1 Oscillator

Commit message: Layout updates
Routing:
- net VCOM: track 43.3 -> 72.4 mm
- net GND: track 139.3 -> 140.3 mm, vias 46 -> 47
Other:
- board text added: "AC Rev 1.0"
